File: dp-to-pcie/dp-to-pcie.sch (KiCad schematic (older format))
At the start: 0 parts

Commit message: Updates to the dp-to-pcie schematic.
Parts:
- added DRX1, DTX1: DISPLAY_PORT, symbol DISPLAY_PORT
- added P?: CONN_02X04, symbol CONN_02X04
- added SW?: SW_PUSH_SMALL, symbol SW_PUSH_SMALL
- added U?: TIMVIDEOS-PCIE-8X, symbol TIMVIDEOS-PCIE-8X
Connections:
- net labels added: DRX0_N, DRX0_P, DRX1_N, DRX1_P, DRX2_N, DRX2_P, DRX3_N, DRX3_P, EXTCLK_N, EXTCLK_P, ~RST
- wire segments 0 -> 125
