File: dp-aux-intercept/dp-aux-intercept.sch (KiCad schematic (older format))
At the start: 24 parts

Commit message: Temp commit.
Connections:
- net JDCFG1: now reaches JDCFG1.4 (P4), RDCFG1.2
- net JDCFG2: now reaches JDCFG1.6 (P6), RDCFG2.2
- net JDHPD: now reaches JDCFG1.2 (P2), RDHPD1.2
- net JCCFG1: now reaches JCCFG1.4 (P4), RCCFG1.2
- net JCCFG2: now reaches JCCFG1.6 (P6), RCCFG2.2
- net JCHPD: now reaches JCCFG1.2 (P2), RCHPD1.2
Changed lines of the file:
@@
 	5070 4940 5290 4940
 Wire Wire Line
-	5290 4940 5290 5130
-Wire Wire Line
-	5290 5130 4820 5130
-Wire Wire Line
-	4820 5130 4350 5130
+	5290 5130 5290 4940
+Wire Wire Line
+	4350 5130 4820 5130
+Wire Wire Line
+	4820 5130 5290 5130
 Wire Wire Line
 	1940 2640 2480 2640
@@
 	6070 2820 6230 2820
 Wire Wire Line
-	6070 2920 6140 2920
-Wire Wire Line
-	6140 2920 6140 2990
-Wire Wire Line
-	6140 2990 6230 2990
+	6070 2920 6160 2920
+Wire Wire Line
+	6160 2920 6160 2990
+Wire Wire Line
+	6160 2990 6230 2990
 Wire Wire Line
 	5540 2340 5540 2720
@@
 Connection ~ 2970 2990
 Wire Wire Line
-	3500 2820 3340 2820
-Wire Wire Line
-	3500 2920 3430 2920
-Wire Wire Line
 	3430 2920 3430 2990
 Wire Wire Line
@@
 	2750 2340 2750 2940
 Wire Wire Line
-	5290 2740 5290 2930
-Wire Wire Line
-	5290 2930 4810 2930
-Wire Wire Line
-	4810 2930 4340 2930
+	5290 2930 5290 2740
+Wire Wire Line
+	4340 2930 4810 2930
+Wire Wire Line
+	4810 2930 5290 2930
 Wire Wire Line
 	4340 2930 4340 2740
@@
 Connection ~ 2970 2820
 Wire Wire Line
-	3350 2650 3440 2650
-Wire Wire Line
-	3440 2650 3440 2720
-Wire Wire Line
-	3440 2720 3500 2720
+	3350 2650 3430 2650
+Wire Wire Line
+	3430 2650 3430 2720
 Wire Wire Line
 	4000 2720 4040 2720
@@
 Wire Wire Line
 	6160 2650 6230 2650
+Wire Wire Line
+	3500 2920 3430 2920
+Wire Wire Line
+	3500 2820 3340 2820
+Wire Wire Line
+	3430 2720 3500 2720
+Text Label 3440 2720 0    10   ~ 0
+JCHPD
+Text Label 3440 2820 0    10   ~ 0
+JCCFG1
+Text Label 3440 2920 0    10   ~ 0
+JCCFG2
+Text Label 6100 2720 0    10   ~ 0
+JDHPD
+Text Label 6090 2820 0    10   ~ 0
+JDCFG1
+Text Label 6090 2920 0    10   ~ 0
+JDCFG2
 $EndSCHEMATC
